File: eda files/explorer-robot/rgb_led.kicad_sch (KiCad schematic)
At the start: 4 parts, among them J5 Conn_01x04

Commit message: Add LiDAR power and UART interface
Add a new lidar schematic sheet with a 4-pin connector, an
AO3400A low-side MOSFET for power switching, and gate pull
resistors. Wire LIDAR_PWR, LIDAR_TX, and LIDAR_RX hierarchical
labels into the MCU sheet and update designators.

Also shorten connector value labels to BAT, LED, and MBR.
Parts:
- J5: value Conn_01x04 -> LED
Changed lines of the file:
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@@
 			)
 		)
-		(property "Value" "Conn_01x04"
+		(property "Value" "LED"
 			(at 163.83 101.5999 0)
 			(show_name no)
