File: eda files/explorer-robot/rp2354b.kicad_sch (KiCad schematic)
At the start: 34 parts, among them J1 DBG, SW1 SW_Push, U1 RP2354B, U2 AMS1117-3.3, Y1 ABM8-272-T3

Commit message: ``` Move AI camera branch to 3.3 V rail
The Grove Vision AI V2 module used here requires a 3.3 V input,
so powering it from the switched 5 V branch would over-voltage it.
Point U9 VIN at +3.3V; the TPS22917, footprint and control are
unchanged.

Also bump the 5 V inductor to 15 µH/3 A, swap the catch diode,
clean up schematic wiring and add no-connects on unused pins.
Document the decision in ADR-0025 and update ADR-0019, ADR-0021
and CONTEXT.md.
```
Connections:
- no-connect marks 0 -> 8
Changed lines of the file:
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@@
 		(color 0 0 0 0)
+	)
+	(no_connect
+		(at 148.59 148.59)
+	)
+	(no_connect
+		(at 146.05 148.59)
+	)
+	(no_connect
+		(at 153.67 148.59)
+	)
+	(no_connect
+		(at 133.35 148.59)
+	)
+	(no_connect
+		(at 151.13 148.59)
+	)
+	(no_connect
+		(at 143.51 148.59)
+	)
+	(no_connect
+		(at 140.97 148.59)
+	)
+	(no_connect
+		(at 130.81 148.59)
 	)
 	(wire

Commit message: Add rear rangefinder to schematic and docs
Document the rear VL53L0X module as a second floor-drop sensor on
I2C1. Add ADR-0026 covering the two unswitched 3.3 V connectors, their
XSHUT/INT GPIO assignments (1-3, 31), pull-ups and series resistors,
and the new rangefinders schematic sheet. Amend ADR-0021, ADR-0022 and
ADR-0024 to note the GPIOs are no longer spare, and update CONTEXT,
README and firmware docs to describe the front/rear pair.
Connections:
- net RF_REAR_INT: now reaches U1.39 (GPIO31)
- net RF_FRONT_XSHUT: now reaches U1.78 (GPIO1)
- net RF_FRONT_INT: now reaches U1.79 (GPIO2)
- net RF_REAR_XSHUT: now reaches U1.80 (GPIO3)
Changed lines of the file:
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@@
+	(wire
+		(pts
+			(xy 115.57 95.25) (xy 115.57 97.79)
+		)
+		(stroke
+			(width 0)
+			(type default)
+		)
+	)
 	(wire
 		(pts
@@
 	(wire
 		(pts
+			(xy 110.49 95.25) (xy 110.49 97.79)
+		)
+		(stroke
+			(width 0)
+			(type default)
+		)
+	)
+	(wire
+		(pts
 			(xy 218.44 38.1) (xy 220.98 38.1)
 		)
@@
 	(wire
 		(pts
+			(xy 113.03 95.25) (xy 113.03 97.79)
+		)
+		(stroke
+			(width 0)
+			(type default)
+		)
+	)
+	(wire
+		(pts
 			(xy 140.97 95.25) (xy 140.97 97.79)
 		)
@@
 		(pts
 			(xy 168.91 95.25) (xy 168.91 97.79)
+		)
+		(stroke
+			(width 0)
+			(type default)
+		)
+	)
+	(wire
+		(pts
+			(xy 186.69 95.25) (xy 186.69 97.79)
 		)
 		(stroke
@@
 		)
 	)
+	(hierarchical_label "RF_FRONT_XSHUT"
+		(shape output)
+		(at 110.49 95.25 90)
+		(effects
+			(font
+				(size 1.27 1.27)
+			)
+			(justify left)
+		)
+	)
 	(hierarchical_label "EXP_RX"
 		(shape input)
@@
 		)
 	)
+	(hierarchical_label "RF_FRONT_INT"
+		(shape input)
+		(at 113.03 95.25 90)
+		(effects
+			(font
+				(size 1.27 1.27)
+			)
+			(justify left)
+		)
+	)
 	(hierarchical_label "LCD_DC"
 		(shape output)
@@
 		)
 	)
+	(hierarchical_label "RF_REAR_XSHUT"
+		(shape output)
+		(at 115.57 95.25 90)
+		(effects
+			(font
+				(size 1.27 1.27)
+			)
+			(justify left)
+		)
+	)
 	(hierarchical_label "AICAM_TX"
 		(shape input)
@@
 		(effects
 			(font
+				(size 1.27 1.27)
+			)
+			(justify left)
+		)
+	)
+	(hierarchical_label "RF_REAR_INT"
+		(shape input)
+		(at 186.69 95.25 90)
+		(effects
+			(font

Commit message: place test points, tidy up, ERC
Parts:
- removed TP5: T.SPI0.CLK, tp:TestPoint_Bridge_Pitch3.81mm_Drill1.3mm, symbol Connector:TestPoint_2Pole
- removed TP6: T.SPI0.MOSI, tp:TestPoint_Bridge_Pitch3.81mm_Drill1.3mm, symbol Connector:TestPoint_2Pole
- removed TP7: T.SPI0.MISO, tp:TestPoint_Bridge_Pitch3.81mm_Drill1.3mm, symbol Connector:TestPoint_2Pole
- added TP14: T.SPI0.CLK, Connector_PinHeader_2.54mm:PinHeader_1x02_P2.54mm_Vertical, symbol Connector:TestPoint_2Pole
- added TP15: T.SPI0.MOSI, Connector_PinHeader_2.54mm:PinHeader_1x02_P2.54mm_Vertical, symbol Connector:TestPoint_2Pole
- added TP16: T.SPI0.MISO, Connector_PinHeader_2.54mm:PinHeader_1x02_P2.54mm_Vertical, symbol Connector:TestPoint_2Pole
- added TP17: T.SPI1.CLK, Connector_PinHeader_2.54mm:PinHeader_1x02_P2.54mm_Vertical, symbol Connector:TestPoint_2Pole
- added TP18: T.SPI1.MOSI, Connector_PinHeader_2.54mm:PinHeader_1x02_P2.54mm_Vertical, symbol Connector:TestPoint_2Pole
- added TP19: T.SPI1.MISO, Connector_PinHeader_2.54mm:PinHeader_1x02_P2.54mm_Vertical, symbol Connector:TestPoint_2Pole
- added TP23: T.PWR.1V1, Connector_PinHeader_2.54mm:PinHeader_1x02_P2.54mm_Vertical, symbol Connector:TestPoint_2Pole
- added TP26: T.I2C1.SDA, Connector_PinHeader_2.54mm:PinHeader_1x02_P2.54mm_Vertical, symbol Connector:TestPoint_2Pole
- added TP27: T.I2C1.SCL, Connector_PinHeader_2.54mm:PinHeader_1x02_P2.54mm_Vertical, symbol Connector:TestPoint_2Pole
- added TP28: T.I2C0.SDA, Connector_PinHeader_2.54mm:PinHeader_1x02_P2.54mm_Vertical, symbol Connector:TestPoint_2Pole
- added TP29: T.I2C0.SCL, Connector_PinHeader_2.54mm:PinHeader_1x02_P2.54mm_Vertical, symbol Connector:TestPoint_2Pole
- TP1, TP2: footprint tp:TestPoint_Bridge_Pitch3.81mm_Drill1.3mm -> Connector_PinHeader_2.54mm:PinHeader_1x02_P2.54mm_Vertical
- Y1: footprint Crystal:Crystal_SMD_Abracon_ABM8AIG-4Pin_3.2x2.5mm -> easyeda imports:CRYSTAL-SMD_4P-L3.2-W2.5-BL
Connections:
- net +1V1: now also TP23.2
- net GND: now also TP14.1, TP15.1, TP16.1, TP17.1, TP18.1, TP19.1, TP23.1, TP26.1, TP27.1, TP28.1, TP29.1
- net I2C0_SCL: now also TP29.2
- net I2C0_SDA: now also TP28.2
- net I2C1_SCL: now also TP27.2
- net I2C1_SDA: now also TP26.2
- net ICM-20948_SCLK: now also TP14.2
- net ICM-20948_SDI: now also TP15.2
- net ICM-20948_SDO: now also TP16.2
- net SPI1_MISO: now also TP19.2
- net SPI1_MOSI: now also TP18.2
- net SPI1_SCK: now also TP17.2
Other:
- note added: "Test Points"
- moved on the sheet: C1, C2, C3, J1, L1, R1, U1
