File: eda files/explorer-robot/rangefinders.kicad_sch (KiCad schematic)
At the start: 14 parts, among them J13 RF.FRONT, J14 RF.REAR

Commit message: Add LCSC part metadata to explorer-robot schematics
Populate JLCPCB_URL, LCSC, MPN, and MFR fields on components in the
panel and rangefinder sheets, and default the BOM view to sort by
LCSC ascending. Rename TB6612FNG test points to match motor encoder
nets, adjust their placement, and drop two symbols from the BOM and
position files.
Parts:
- C63, C65: JLCPCB_URL (none) -> https://jlcpcb.com/partdetail/16532-CL21A106KAYNNNE/C15850; LCSC (none) -> C15850; MFR (none) -> Samsung Electro-Mechanics; MPN (none) -> CL21A106KAYNNNE
- C64, C66: JLCPCB_URL (none) -> https://jlcpcb.com/partdetail/YAGEO-CC0603KRX7R9BB104/C14663; LCSC (none) -> C14663; MFR (none) -> YAGEO; MPN (none) -> CC0603KRX7R9BB104
- J13, J14: now left out of the parts list
- R37, R38, R41, R42: JLCPCB_URL (none) -> https://jlcpcb.com/partdetail/23867-0603WAF330JT5E/C23140; LCSC (none) -> C23140; MPN (none) -> 0603WAF330JT5E
- R39, R40, R43, R44: JLCPCB_URL (none) -> https://jlcpcb.com/partdetail/23889-0603WAF4701T5E/C23162; LCSC (none) -> C23162

Commit message: Update AI camera branch to 5V and document schematic
- ADR-0027 supersedes ADR-0025: AI camera input is 5V, not 3.3V
- Move U9 VIN and C55 back to +5V in aicam.kicad_sch
- Update CONTEXT.md branch descriptions and ADR cross-references
- Record ICM-20948 placement status and corrected battery divider ratio
- Adjust battery_charge_read for 33k/10k divider (0.2326 ratio)
- Enable sheet component classes; refresh netlist and PCB footprints
Parts:
- R37, R38, R41, R42: MFR (none) -> UNI-ROYAL(Uniroyal Elec)
Changed lines of the file:
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@@
+			)
+		)
+		(property "MFR" "UNI-ROYAL(Uniroyal Elec)"
+			(at 67.31 99.06 90)
+			(hide yes)
+			(show_name no)
+			(do_not_autoplace no)
+			(effects
+				(font
+					(size 1.27 1.27)
+				)
 			)
 		)
@@
 			)
 		)
+		(property "MFR" "UNI-ROYAL(Uniroyal Elec)"
+			(at 176.53 99.06 90)
+			(hide yes)
+			(show_name no)
+			(do_not_autoplace no)
+			(effects
+				(font
+					(size 1.27 1.27)
+				)
+			)
+		)
 		(pin "1"
 		)
@@
 			)
 		)
+		(property "MFR" "UNI-ROYAL(Uniroyal Elec)"
+			(at 67.31 101.6 90)
+			(hide yes)
+			(show_name no)
+			(do_not_autoplace no)
+			(effects
+				(font
+					(size 1.27 1.27)
+				)
+			)
+		)
 		(pin "1"
 		)
@@
 			(at 176.53 101.6 90)
 			(hide yes)
+			(show_name no)
+			(do_not_autoplace no)
+			(effects
+				(font
+					(size 1.27 1.27)
+				)
+			)
+		)
+		(property "MFR" "UNI-ROYAL(Uniroyal Elec)"
+			(at 176.53 101.6 90)
+			(hide yes)
