File: eda files/explorer-robot/tb6612fng.kicad_sch (KiCad schematic)
At the start: 21 parts, among them J2 Motor_A_left, J3 Motor_B_right, U6 TB6612FNG

Commit message: Add ADR-0021 for expansion UART and camera on PIO
Add an RGB LED connector sheet to the schematic.
Other:
- title: (none) -> Motor Driver and Motor/Encoder Connectors
Changed lines of the file:
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@@
 	(paper "A4")
 	(title_block
+		(title "Motor Driver and Motor/Encoder Connectors")
 		(date "2026-09-27")
 		(rev "v.0.1")

Commit message: Add LiDAR power and UART interface
Add a new lidar schematic sheet with a 4-pin connector, an
AO3400A low-side MOSFET for power switching, and gate pull
resistors. Wire LIDAR_PWR, LIDAR_TX, and LIDAR_RX hierarchical
labels into the MCU sheet and update designators.

Also shorten connector value labels to BAT, LED, and MBR.
Parts:
- J2: value Motor_A_left -> MAL
- J3: value Motor_B_right -> MBR
Changed lines of the file:
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@@
 			)
 		)
-		(property "Value" "Motor_B_right"
+		(property "Value" "MBR"
 			(at 266.7 106.6799 0)
 			(show_name no)
@@
 			)
 		)
-		(property "Value" "Motor_A_left"
+		(property "Value" "MAL"
 			(at 267.97 45.7199 0)
 			(show_name no)

Commit message: place test points, tidy up, ERC
Parts:
- added TP24: T., Connector_PinHeader_2.54mm:PinHeader_1x02_P2.54mm_Vertical, symbol Connector:TestPoint_2Pole
- added TP25: XYZ, Connector_PinHeader_2.54mm:PinHeader_1x02_P2.54mm_Vertical, symbol Connector:TestPoint_2Pole
- TP10, TP11: footprint tp:TestPoint_Bridge_Pitch3.81mm_Drill1.3mm -> Connector_PinHeader_2.54mm:PinHeader_1x02_P2.54mm_Vertical
Connections:
- net GND: now also TP24.1, TP25.1
- net MOT.A.L.ENC.A: now also TP24.2
- net MOT.B.R.ENC.A: now also TP25.2
Other:
- note removed: "If board space is too tight these test points might be dropped: Testing motor signals should be possible at the connector, too."
- moved on the sheet: TP10, TP11

Commit message: Add LCSC part metadata to explorer-robot schematics
Populate JLCPCB_URL, LCSC, MPN, and MFR fields on components in the
panel and rangefinder sheets, and default the BOM view to sort by
LCSC ascending. Rename TB6612FNG test points to match motor encoder
nets, adjust their placement, and drop two symbols from the BOM and
position files.
Parts:
- TP24: value T. -> T.MOT.ENC.A
- TP25: value XYZ -> T.MOT.ENC.B
Other:
- moved on the sheet: TP10, TP25
Changed lines of the file:
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@@
 	(wire
 		(pts
-			(xy 26.67 36.83) (xy 29.21 36.83)
+			(xy 26.67 35.56) (xy 29.21 35.56)
 		)
 		(stroke
@@
 	(wire
 		(pts
-			(xy 39.37 36.83) (xy 41.91 36.83)
+			(xy 39.37 35.56) (xy 41.91 35.56)
 		)
 		(stroke
@@
 	(wire
 		(pts
-			(xy 39.37 52.07) (xy 41.91 52.07)
+			(xy 39.37 53.34) (xy 41.91 53.34)
 		)
 		(stroke
@@
 	(wire
 		(pts
-			(xy 26.67 52.07) (xy 29.21 52.07)
+			(xy 26.67 53.34) (xy 29.21 53.34)
 		)
 		(stroke
@@
 	)
 	(label "B02"
-		(at 41.91 36.83 0)
+		(at 41.91 35.56 0)
 		(effects
 			(font
@@
 	)
 	(label "B01"
-		(at 26.67 36.83 180)
+		(at 26.67 35.56 180)
 		(effects
 			(font
@@
 	(hierarchical_label "MOT.B.R.ENC.A"
 		(shape output)
-		(at 41.91 52.07 0)
+		(at 41.91 53.34 0)
 		(effects
 			(font
@@
 			)
 		)
-		(property "Value" "T."
+		(property "Value" "T.MOT.ENC.A"
 			(at 34.29 41.91 0)
 			(show_name no)
@@
 	(symbol
 		(lib_id "Connector:TestPoint_2Pole")
-		(at 34.29 52.07 0)
+		(at 34.29 53.34 0)
 		(unit 1)
 		(body_style 1)
@@
 		(fields_autoplaced yes)
 		(property "Reference" "TP25"
-			(at 34.29 46.99 0)
+			(at 34.29 48.26 0)
 			(show_name no)
 			(do_not_autoplace no)
@@
 			)
 		)
-		(property "Value" "XYZ"
-			(at 34.29 49.53 0)
+		(property "Value" "T.MOT.ENC.B"
+			(at 34.29 50.8 0)
 			(show_name no)
 			(do_not_autoplace no)
@@
 		)
 		(property "Footprint" "Connector_PinHeader_2.54mm:PinHeader_1x02_P2.54mm_Vertical"
-			(at 34.29 52.07 0)
+			(at 34.29 53.34 0)
 			(hide yes)
 			(show_name no)
@@
 		)
 		(property "Datasheet" ""
-			(at 34.29 52.07 0)
+			(at 34.29 53.34 0)
 			(hide yes)
 			(show_name no)
@@
 		)
 		(property "Description" "2-polar test point"
-			(at 34.29 52.07 0)
+			(at 34.29 53.34 0)
 			(hide yes)
 			(show_name no)
@@
 		)
 		(property "JLCPCB_URL" ""
-			(at 34.29 52.07 0)
+			(at 34.29 53.34 0)
 			(hide yes)
 			(show_name no)
@@
 		)
 		(property "KLC_S3.3" ""
-			(at 34.29 52.07 0)
+			(at 34.29 53.34 0)
 			(hide yes)
 			(show_name no)
@@
 		)
 		(property "KLC_S4.1" ""
-			(at 34.29 52.07 0)
+			(at 34.29 53.34 0)
 			(hide yes)
 			(show_name no)
@@
 		)
 		(property "KLC_S4.2_DVDD" ""
-			(at 34.29 52.07 0)
+			(at 34.29 53.34 0)
 			(hide yes)
 			(show_name no)
@@
 		)
 		(property "KLC_S4.2_VREG_LX" ""
-			(at 34.29 52.07 0)
+			(at 34.29 53.34 0)
 			(hide yes)
 			(show_name no)
@@
 		)
 		(property "MFR" ""
-			(at 34.29 52.07 0)
+			(at 34.29 53.34 0)
 			(hide yes)
 			(show_name no)
@@
 		)
 		(property "JLCPCP_URL" ""
-			(at 34.29 52.07 0)
+			(at 34.29 53.34 0)
 			(hide yes)
 			(show_name no)
@@
 	(symbol
 		(lib_id "power:GND")
-		(at 26.67 52.07 270)
+		(at 26.67 53.34 270)
 		(unit 1)
 		(body_style 1)
@@
 		(fields_autoplaced yes)
 		(property "Reference" "#PWR0119"
-			(at 20.32 52.07 0)
+			(at 20.32 53.34 0)
 			(hide yes)
 			(show_name no)
@@
 		)
 		(property "Value" "GND"
-			(at 22.86 52.0699 90)
+			(at 22.86 53.3399 90)
 			(show_name no)
 			(do_not_autoplace no)
@@
 		)
 		(property "Footprint" ""
-			(at 26.67 52.07 0)
+			(at 26.67 53.34 0)
 			(hide yes)
 			(show_name no)
@@
 		)
 		(property "Datasheet" ""
-			(at 26.67 52.07 0)
+			(at 26.67 53.34 0)
 			(hide yes)
 			(show_name no)
@@
 		)
 		(property "Description" "Power symbol creates a global label with name \"GND\" , ground"
-			(at 26.67 52.07 0)
+			(at 26.67 53.34 0)
 			(hide yes)
 			(show_name no)
@@
 	(symbol
 		(lib_id "Connector:TestPoint_2Pole")
-		(at 34.29 36.83 0)
+		(at 34.29 35.56 0)
 		(unit 1)
 		(body_style 1)
@@
 		(fields_autoplaced yes)
 		(property "Reference" "TP10"
-			(at 34.29 31.75 0)
+			(at 34.29 30.48 0)
 			(show_name no)
 			(do_not_autoplace no)
@@
 		)
 		(property "Value" "T.MOT.B"
-			(at 34.29 34.29 0)
+			(at 34.29 33.02 0)
 			(show_name no)
 			(do_not_autoplace no)
@@
 		)
 		(property "Footprint" "Connector_PinHeader_2.54mm:PinHeader_1x02_P2.54mm_Vertical"
-			(at 34.29 36.83 0)
+			(at 34.29 35.56 0)
 			(hide yes)
 			(show_name no)
@@
 		)
 		(property "Datasheet" ""
-			(at 34.29 36.83 0)
+			(at 34.29 35.56 0)
 			(hide yes)
 			(show_name no)
@@
 		)
 		(property "Description" "2-polar test point"
-			(at 34.29 36.83 0)
+			(at 34.29 35.56 0)
 			(hide yes)
 			(show_name no)
@@
 		)
 		(property "JLCPCB_URL" ""
-			(at 34.29 36.83 0)
+			(at 34.29 35.56 0)
 			(hide yes)
 			(show_name no)
@@
 		)
 		(property "KLC_S3.3" ""
-			(at 34.29 36.83 0)
+			(at 34.29 35.56 0)
 			(hide yes)
 			(show_name no)
@@
 		)
 		(property "KLC_S4.1" ""
-			(at 34.29 36.83 0)
+			(at 34.29 35.56 0)
 			(hide yes)
 			(show_name no)
@@
 		)
 		(property "KLC_S4.2_DVDD" ""
-			(at 34.29 36.83 0)
+			(at 34.29 35.56 0)
 			(hide yes)
 			(show_name no)
@@
 		)
 		(property "KLC_S4.2_VREG_LX" ""
-			(at 34.29 36.83 0)
+			(at 34.29 35.56 0)
 			(hide yes)
 			(show_name no)
@@
 		)
 		(property "MFR" ""
-			(at 34.29 36.83 0)
+			(at 34.29 35.56 0)
 			(hide yes)
 			(show_name no)
@@
 		)
 		(property "JLCPCP_URL" ""
-			(at 34.29 36.83 0)
+			(at 34.29 35.56 0)
 			(hide yes)
 			(show_name no)

Commit message: Change TB6612FNG bypass caps to 2n2 and note TXB0108 grounding
- Swap two 10n capacitors for 2n2 (LCSC C1604) in the TB6612FNG
  schematic
- Change BOM sort field from Reference to Value
- Document tying unused TXB0108 I/O pairs to GND in ADR 0017
Parts:
- C32: value 10n -> 2n2; JLCPCB_URL https://jlcpcb.com/partdetail/58143-0603B103K500NT/C57112 -> https://jlcpcb.com/partdetail/1956-0603B222K500NT/C1604; LCSC C57112 -> C1604; MPN 0603B103K500NT -> 0603B222K500NT
- C34: value 10n -> 2n2; JLCPCB_URL https://jlcpcb.com/partdetail/58143-0603B103K500NT/C57112 -> https://jlcpcb.com/partdetail/1956-0603B222K500NT/C1604; JLCPCP_URL (none) -> https://jlcpcb.com/partdetail/1956-0603B222K500NT/C1604; LCSC C57112 -> C1604; MPN 0603B103K500NT -> 0603B222K500NT
Changed lines of the file:
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@@
 			)
 		)
-		(property "Value" "10n"
+		(property "Value" "2n2"
 			(at 238.506 121.666 0)
 			(show_name no)
@@
 			)
 		)
-		(property "MPN" "0603B103K500NT"
+		(property "MPN" "0603B222K500NT"
 			(at 237.49 119.38 0)
 			(hide yes)
@@
 			)
 		)
-		(property "LCSC" "C57112"
+		(property "LCSC" "C1604"
 			(at 237.49 119.38 0)
 			(hide yes)
@@
 			)
 		)
-		(property "JLCPCB_URL" "https://jlcpcb.com/partdetail/58143-0603B103K500NT/C57112"
+		(property "JLCPCB_URL" "https://jlcpcb.com/partdetail/1956-0603B222K500NT/C1604"
 			(at 237.49 119.38 0)
 			(hide yes)
@@
 			)
 		)
-		(property "JLCPCP_URL" ""
+		(property "JLCPCP_URL" "https://jlcpcb.com/partdetail/1956-0603B222K500NT/C1604"
 			(at 237.49 119.38 0)
 			(hide yes)
@@
 			)
 		)
-		(property "Value" "10n"
+		(property "Value" "2n2"
 			(at 239.776 61.976 0)
 			(show_name no)
@@
 			)
 		)
-		(property "MPN" "0603B103K500NT"
+		(property "MPN" "0603B222K500NT"
 			(at 238.76 59.69 0)
 			(hide yes)
@@
 			)
 		)
-		(property "LCSC" "C57112"
+		(property "LCSC" "C1604"
 			(at 238.76 59.69 0)
 			(hide yes)
@@
 			)
 		)
-		(property "JLCPCB_URL" "https://jlcpcb.com/partdetail/58143-0603B103K500NT/C57112"
+		(property "JLCPCB_URL" "https://jlcpcb.com/partdetail/1956-0603B222K500NT/C1604"
 			(at 238.76 59.69 0)
 			(hide yes)
